File: Daring Maimu-Leelo.brd (EAGLE design)
At the start: 218.8 x 67.8 mm, 17 parts, among them U1 ARDUINO-UNO-R3-SHIELD

Commit message: Updated code acording to new requests from the professor 	-Still need to check if the 7segment display is working but cant 	do to the stupidity of a certain someone Updated the circuit to acomodate the new request from the professor 	-Still need to check if its working
Parts:
- removed DIGIT1: 7SEG-CA, Tinkercad:7SEG-13
- removed PIEZO1: PIEZO, Tinkercad:PIEZO
- added DIGIT2: 7SEG-CA, Tinkercad:7SEG-13
- added R10, R11, R12, R13, R14, R17, R18, R19, R20, R8, R9: 1k, Tinkercad:RESAD1016W63L850D250B
- added U2: CD4511_PDIP, Tinkercad:DIP762W53P254L1969H508Q16B
- moved R6 31.0 mm to (129.9, 41.6)
- moved S1 31.0 mm to (109.6, 53.0)
- moved S2 31.0 mm to (124.8, 53.0)
- moved D1 31.0 mm to (88.0, 39.1)
- moved D2 31.0 mm to (95.6, 39.1)
- moved D3 31.0 mm to (103.2, 39.1)
- moved D4 31.0 mm to (156.6, 59.4)
- moved R1 31.0 mm to (96.9, 51.8)
- moved R2 31.0 mm to (117.2, 46.7)
- moved R3 31.0 mm to (136.3, 46.7)
- moved R4 31.0 mm to (89.3, 51.8)
- moved R5 31.0 mm to (104.5, 51.8)
- moved R7 31.0 mm to (157.8, 51.8)
- moved U1 31.0 mm to (47.9, 69.0)
- moved DIST1 31.0 mm to (149.0, 67.0)
Connections:
- removed net U1_A1: R4.2, U1.A1
- removed net U1_A2: R1.2, U1.A2
- removed net U1_A3: R5.2, U1.A3
- removed net U1_RX: DIGIT1.1, U1.RX
- removed net U1_TX: DIGIT1.4, U1.TX
- new net DIGIT2_A: DIGIT2.7, R13.2
- new net DIGIT2_B: DIGIT2.6, R14.1
- new net DIGIT2_C: DIGIT2.4, R10.1
- new net DIGIT2_D: DIGIT2.2, R9.1
- new net DIGIT2_E: DIGIT2.1, R8.1
- new net DIGIT2_F: DIGIT2.9, R12.2
- new net DIGIT2_G: DIGIT2.10, R11.1
- new net U1_D12: R19.2, U1.D12
- new net U2_A: R13.1, U2.13
- new net U2_B: R14.2, U2.12
- new net U2_C: R10.2, U2.11
- new net U2_D: R9.2, U2.10
- new net U2_E: R8.2, U2.9
- new net U2_F: R11.2, U2.15
- new net U2_G: R12.1, U2.14
- new net U2_IA: R17.1, U2.7
- new net U2_IB: R20.1, U2.1
- new net U2_IC: R19.1, U2.2
- new net U2_ID: R18.1, U2.6
- net U1_5V: no longer R3.2
- net U1_D10: now also R18.2; no longer DIGIT1.7
- net U1_D13: now also R20.2; no longer PIEZO1.1
- net U1_D5: now also R3.2, U2.8; no longer DIGIT1.8, PIEZO1.2
- net U1_D6: now also R4.2; no longer DIGIT1.6
- net U1_D7: now also R1.2; no longer DIGIT1.9
- net U1_D8: now also R5.2; no longer DIGIT1.10
- net U1_D9: now also R17.2; no longer DIGIT1.2
Other:
- board size 218.8 x 67.8 mm -> 241.3 x 106.6 mm
